File: PCB/Proyecto_Kicad/estapa_de_control.kicad_pcb (KiCad board)
At the start: 2 copper layers, 149 x 119 mm, 70 parts, among them K1 SANYOU_SRD_Form_C, K2 SANYOU_SRD_Form_C, K3 SANYOU_SRD_Form_C, Q1 BC548, Q10 BC548, Q11 BC548, Q12 BC548, Q13 BC548, Q2 BC548, Q3 BC548, Q4 BC548, Q5 BC548, Q6 BC548, Q7 BC548, Q8 BC548, Q9 BC548, U1 RP2040-Zero, U2 ESP-01v090

Commit message: fix: "Corrección de errores de la placa"
Parts:
- removed the GraviCap at (135.0, 86.0)
- removed the R1 at (140.7, 72.5)
- added GraviCap: LOGO, LOGO, F.Cu at (135.1, 92.0)
- D2: renamed from D4; footprint Diode_THT:D_A-405_P10.16mm_Horizontal -> Diode_THT:D_5W_P10.16mm_Horizontal
- moved D4 28.6 mm to (149.0, 120.9), turned to -90 degrees
- moved D3 19.3 mm to (201.1, 122.0), turned to 180 degrees
- moved K2 16.0 mm to (154.5, 125.0), turned to 0 degrees
- moved R25 11.5 mm to (189.6, 21.0), turned to 0 degrees
- moved K1 1.00 mm to (187.0, 115.5)
- renumbered 0X45_Entrega_panel_solar1 to 0X41_MPPT1, 0X41_MPPT1 to 0X45_Panel_Solar1, D3 to D1, D1 to D3, D5 to D4, D2 to D5, K3 to K2, K2 to K3, LED_Amarillo_2 to LED_Amarillo_1, LED_Amarillo_1 to LED_Amarillo_2, LED_Azul_2 to LED_Azul_1, LED_Azul_3 to LED_Azul_2, LED_Azul_1 to LED_Azul_3, LED_Rojo_2 to LED_Rojo_1, LED_Rojo_1 to LED_Rojo_2, Panel_Solar1 to MPPT1, MPPT1 to Panel_Solar1, Q11 to Q10, Q4 to Q11, Q5 to Q13, Q6 to Q2, Q9 to Q3, Q13 to Q4, Q2 to Q5, Q7 to Q6, Q10 to Q7, Q3 to Q8, Q8 to Q9, R2 to R1, R11 to R10, R19 to R11, R7 to R12, R16 to R13, R22 to R14, R4 to R15, R12 to R16, R20 to R17, R8 to R18, R17 to R19, R10 to R2, R23 to R20, R13 to R21, R24 to R22, R14 to R23, R5 to R24, R9 to R25, R18 to R3, R25 to R4, R6 to R5, R15 to R6, R21 to R7, R26 to R8, R3 to R9, U2 to U1, U1 to U2
Connections:
- net Vin-_Solar renamed Vin-_MPPT
- 0X41_MPPT1 pad 8: Panel_Solar_+ -> MPPT_+
- 0X45_Panel_Solar1 pad 8: MPPT_+ -> Panel_Solar_+
- K2 pad 3: Motor_Vin+ -> unconnected-(K2-Pad3)
- K2 pad 4: unconnected-(K3-Pad4) (its old number) -> Motor_Vin+
- MPPT1 pad 2: Panel_Solar_+ -> MPPT_+
- Panel_Solar1 pad 2: MPPT_+ -> Panel_Solar_+
Routing:
- net +5V: track 455.0 -> 584.3 mm, vias 8 -> 6
- net Panel_Solar_+: track 37.5 -> 91.4 mm
- net MPPT_+: track 91.4 -> 37.5 mm
- net Net-(D4-A): track 72.9 -> 42.2 mm
- net Motor_Vin+: track 139.9 -> 114.2 mm
- net RPZ_LED_6: track 139.6 -> 144.9 mm
- net RPZ_LED_5: track 148.4 -> 153.3 mm
- net RPZ_LED_7: track 134.4 -> 138.5 mm
- net Motor_Vin-: track 62.5 -> 58.4 mm
- net Vin+_Consumo: track 79.7 -> 76.4 mm
- net RPZ_LED_8: track 125.3 -> 128.5 mm
- net RPZ_I2C_SCL: track 159.1 -> 160.4 mm
- net RPZ_LED_9: track 124.5 -> 125.6 mm
- net RPZ_RELE_3: track 11.7 -> 10.7 mm
- net RPZ_RELE_2: track 16.6 -> 15.6 mm
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